Commit message: single object datasets version

File: data/robotiq_85/urdf/ur5_robotiq_85.urdf (robot description, URDF)
Before this commit: robot ur5_robotiq_85, 17 links, 16 joints
Joints:
- joint finger_joint: limit lower=0 upper=0.8 effort=1000 velocity=2.0 -> lower=0 upper=0.8 effort=5000 velocity=2.0
- joint left_inner_finger_joint: limit lower=-0.8757 upper=0 effort=1000 velocity=2.0 -> lower=-0.8757 upper=0 effort=5000 velocity=2.0
- joint left_inner_knuckle_joint: limit lower=0 upper=0.8757 effort=1000 velocity=2.0 -> lower=0 upper=0.8757 effort=5000 velocity=2.0
- joint right_inner_finger_joint: limit lower=-0.8757 upper=0 effort=1000 velocity=2.0 -> lower=-0.8757 upper=0 effort=5000 velocity=2.0
- joint right_inner_knuckle_joint: limit lower=0 upper=0.8757 effort=1000 velocity=2.0 -> lower=0 upper=0.8757 effort=5000 velocity=2.0
- joint right_outer_knuckle_joint: limit lower=0 upper=0.81 effort=1000 velocity=2.0 -> lower=0 upper=0.81 effort=5000 velocity=2.0
